File: 5-12.kicad_pcb (KiCad board)
At the start: 2 copper layers, 266.7 x 95.2 mm, 136 parts, among them SW1 SW_Push, U1 ATmega32U4-AU, Y1 16MHz

Commit message: Added col traces between rows
Routing:
- net Col6: track 0.00 -> 80.1 mm
- net Col5: track 0.00 -> 80.1 mm
- net Col9: track 0.00 -> 76.2 mm
- net Col8: track 0.00 -> 76.2 mm
- net Col7: track 0.00 -> 76.2 mm
- net Col4: track 0.00 -> 76.2 mm
- net Col3: track 0.00 -> 76.2 mm
- net Col2: track 0.00 -> 76.2 mm
- net Col11: track 0.00 -> 76.2 mm
- net Col10: track 0.00 -> 76.2 mm
- net Col1: track 0.00 -> 76.2 mm
- net Col0: track 0.00 -> 76.2 mm
Changed lines of the file:
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@@
     (thickness 1.6)
     (drawings 8)
-    (tracks 117)
+    (tracks 182)
     (zones 0)
     (modules 136)
@@
   (segment (start 148.51199 77.85549) (end 152.13949 77.85549) (width 0.381) (layer F.Cu) (net 71))
   (segment (start 147.30625 75.14375) (end 147.30625 76.64975) (width 0.381) (layer F.Cu) (net 71))
+  (segment (start 17.62125 76.04125) (end 17.62125 95.09125) (width 0.254) (layer B.Cu) (net 72))
+  (segment (start 17.62125 95.09125) (end 17.62125 114.14125) (width 0.254) (layer B.Cu) (net 72))
+  (segment (start 17.62125 114.14125) (end 17.62125 133.19125) (width 0.254) (layer B.Cu) (net 72))
+  (segment (start 17.62125 133.19125) (end 17.62125 152.24125) (width 0.254) (layer B.Cu) (net 72))
+  (segment (start 36.67125 152.24125) (end 36.67125 133.19125) (width 0.254) (layer B.Cu) (net 73))
+  (segment (start 36.67125 133.19125) (end 36.67125 114.14125) (width 0.254) (layer B.Cu) (net 73))
+  (segment (start 36.67125 112.55026) (end 36.67125 95.09125) (width 0.254) (layer B.Cu) (net 73))
+  (segment (start 36.67125 114.14125) (end 36.67125 112.55026) (width 0.254) (layer B.Cu) (net 73))
+  (segment (start 36.67125 95.09125) (end 36.67125 76.04125) (width 0.254) (layer B.Cu) (net 73))
+  (segment (start 55.72125 77.63224) (end 55.72125 95.09125) (width 0.254) (layer B.Cu) (net 74))
+  (segment (start 55.72125 76.04125) (end 55.72125 77.63224) (width 0.254) (layer B.Cu) (net 74))
+  (segment (start 55.72125 96.68224) (end 55.72125 114.14125) (width 0.254) (layer B.Cu) (net 74))
+  (segment (start 55.72125 95.09125) (end 55.72125 96.68224) (width 0.254) (layer B.Cu) (net 74))
+  (segment (start 55.72125 114.14125) (end 55.72125 133.19125) (width 0.254) (layer B.Cu) (net 74))
+  (segment (start 55.72125 133.19125) (end 55.72125 152.24125) (width 0.254) (layer B.Cu) (net 74))
+  (segment (start 74.77125 152.24125) (end 74.77125 133.19125) (width 0.254) (layer B.Cu) (net 75))
+  (segment (start 74.77125 117.056316) (end 74.77125 114.14125) (width 0.254) (layer B.Cu) (net 75))
+  (segment (start 74.77125 133.19125) (end 74.77125 117.056316) (width 0.254) (layer B.Cu) (net 75))
+  (segment (start 74.77125 114.14125) (end 74.77125 95.09125) (width 0.254) (layer B.Cu) (net 75))
+  (segment (start 74.77125 95.09125) (end 74.77125 76.04125) (width 0.254) (layer B.Cu) (net 75))
+  (segment (start 93.82125 77.63224) (end 93.82125 95.09125) (width 0.254) (layer B.Cu) (net 76))
+  (segment (start 93.82125 76.04125) (end 93.82125 77.63224) (width 0.254) (layer B.Cu) (net 76))
+  (segment (start 93.82125 95.09125) (end 93.82125 114.14125) (width 0.254) (layer B.Cu) (net 76))
+  (segment (start 93.82125 114.14125) (end 93.82125 133.19125) (width 0.254) (layer B.Cu) (net 76))
+  (segment (start 93.82125 133.19125) (end 93.82125 152.24125) (width 0.254) (layer B.Cu) (net 76))
+  (segment (start 112.87125 134.78224) (end 112.87125 133.19125) (width 0.254) (layer B.Cu) (net 77))
+  (segment (start 121.271251 143.756185) (end 112.87125 135.356184) (width 0.254) (layer B.Cu) (net 77))
+  (segment (start 121.271251 151.116251) (end 121.271251 143.756185) (width 0.254) (layer B.Cu) (net 77))
+  (segment (start 112.87125 135.356184) (end 112.87125 134.78224) (width 0.254) (layer B.Cu) (net 77))
+  (segment (start 122.39625 152.24125) (end 121.271251 151.116251) (width 0.254) (layer B.Cu) (net 77))
+  (segment (start 112.87125 116.172288) (end 112.87125 114.14125) (width 0.254) (layer B.Cu) (net 77))
+  (segment (start 112.87125 133.19125) (end 112.87125 116.172288) (width 0.254) (layer B.Cu) (net 77))
+  (segment (start 112.87125 114.14125) (end 112.87125 95.09125) (width 0.254) (layer B.Cu) (net 77))
+  (segment (start 112.87125 95.09125) (end 112.87125 76.04125) (width 0.254) (layer B.Cu) (net 77))
+  (segment (start 170.02125 77.63224) (end 170.02125 95.09125) (width 0.254) (layer B.Cu) (net 78))
+  (segment (start 170.02125 76.04125) (end 170.02125 77.63224) (width 0.254) (layer B.Cu) (net 78))
+  (segment (start 170.02125 95.09125) (end 170.02125 114.14125) (width 0.254) (layer B.Cu) (net 78))
+  (segment (start 170.02125 115.73224) (end 170.02125 133.19125) (width 0.254) (layer B.Cu) (net 78))
+  (segment (start 170.02125 114.14125) (end 170.02125 115.73224) (width 0.254) (layer B.Cu) (net 78))
+  (segment (start 170.02125 142.71625) (end 160.49625 152.24125) (width 0.254) (layer B.Cu) (net 78))
+  (segment (start 170.02125 133.19125) (end 170.02125 142.71625) (width 0.254) (layer B.Cu) (net 78))
+  (segment (start 189.07125 152.24125) (end 189.07125 133.19125) (width 0.254) (layer B.Cu) (net 79))
+  (segment (start 189.07125 131.60026) (end 189.07125 114.14125) (width 0.254) (layer B.Cu) (net 79))
+  (segment (start 189.07125 133.19125) (end 189.07125 131.60026) (width 0.254) (layer B.Cu) (net 79))
+  (segment (start 189.07125 114.14125) (end 189.07125 95.09125) (width 0.254) (layer B.Cu) (net 79))
+  (segment (start 189.07125 95.09125) (end 189.07125 76.04125) (width 0.254) (layer B.Cu) (net 79))
+  (segment (start 208.12125 76.04125) (end 208.12125 95.09125) (width 0.254) (layer B.Cu) (net 80))
+  (segment (start 208.12125 96.68224) (end 208.12125 114.14125) (width 0.254) (layer B.Cu) (net 80))
+  (segment (start 208.12125 95.09125) (end 208.12125 96.68224) (width 0.254) (layer B.Cu) (net 80))
+  (segment (start 208.12125 115.73224) (end 208.12125 133.19125) (width 0.254) (layer B.Cu) (net 80))
+  (segment (start 208.12125 114.14125) (end 208.12125 115.73224) (width 0.254) (layer B.Cu) (net 80))
+  (segment (start 208.12125 133.19125) (end 208.12125 152.24125) (width 0.254) (layer B.Cu) (net 80))
+  (segment (start 227.17125 152.24125) (end 227.17125 133.19125) (width 0.254) (layer B.Cu) (net 81))
+  (segment (start 227.17125 133.19125) (end 227.17125 114.14125) (width 0.254) (layer B.Cu) (net 81))
+  (segment (start 227.17125 114.14125) (end 227.17125 95.09125) (width 0.254) (layer B.Cu) (net 81))
+  (segment (start 227.17125 95.09125) (end 227.17125 76.04125) (width 0.254) (layer B.Cu) (net 81))
+  (segment (start 246.22125 77.63224) (end 246.22125 95.09125) (width 0.254) (layer B.Cu) (net 82))
+  (segment (start 246.22125 76.04125) (end 246.22125 77.63224) (width 0.254) (layer B.Cu) (net 82))
+  (segment (start 246.22125 95.09125) (end 246.22125 114.14125) (width 0.254) (layer B.Cu) (net 82))
+  (segment (start 246.22125 114.14125) (end 246.22125 133.19125) (width 0.254) (layer B.Cu) (net 82))
+  (segment (start 246.22125 133.19125) (end 246.22125 152.24125) (width 0.254) (layer B.Cu) (net 82))
+  (segment (start 265.27125 76.04125) (end 265.27125 95.09125) (width 0.254) (layer B.Cu) (net 83))
+  (segment (start 265.27125 95.09125) (end 265.27125 114.14125) (width 0.254) (layer B.Cu) (net 83))
+  (segment (start 265.27125 114.14125) (end 265.27125 133.19125) (width 0.254) (layer B.Cu) (net 83))
+  (segment (start 265.27125 133.19125) (end 265.27125 152.24125) (width 0.254) (layer B.Cu) (net 83))
   (segment (start 146.50625 77.49675) (end 147.193 78.1835) (width 0.254) (layer F.Cu) (net 84))
   (segment (start 146.50625 75.14375) (end 146.50625 77.49675) (width 0.254) (layer F.Cu) (net 84))
