File: 5-12.sch (KiCad schematic (older format))
At the start: 136 parts, among them SW1 SW_Push, U1 ATmega32U4-AU, Y1 16MHz

Commit message: Genned production files, made zip
Connections:
- net Row5 is gone; now on net Row4: D10.1 (K), D15.1 (K), D20.1 (K), D25.1 (K), D30.1 (K), D35.1 (K), D40.1 (K), D45.1 (K), D5.1 (K), D50.1 (K), D55.1 (K), D60.1 (K)
- net Col0: now also U1.8 (PB0)
- net Col1: now also U1.9 (PB1)
- net Col10: now also U1.40 (PF1)
- net Col11: now also U1.41 (PF0)
- net Col2: now also U1.10 (PB2)
- net Col3: now also U1.11 (PB3)
- net Col4: now also U1.12 (PB7)
- net Col5: now also U1.18 (PD0)
- net Col6: now also U1.36 (PF7)
- net Col7: now also U1.37 (PF6)
- net Col8: now also U1.38 (PF5)
- net Col9: now also U1.39 (PF4)
- net Row0: now also U1.25 (PD4)
- net Row1: now also U1.26 (PD6)
- net Row2: now also U1.27 (PD7)
- net Row3: now also U1.28 (PB4)
- net Row4: now reaches U1.29 (PB5)
Changed lines of the file:
@@
 Row3
 Text GLabel 4400 4500 0    50   Input ~ 0
-Row5
+Row4
+Text GLabel 3100 1700 2    50   Input ~ 0
+Col0
+Text GLabel 3100 1800 2    50   Input ~ 0
+Col1
+Text GLabel 3100 1900 2    50   Input ~ 0
+Col2
+Text GLabel 3100 2000 2    50   Input ~ 0
+Col3
+Text GLabel 3100 2400 2    50   Input ~ 0
+Col4
+Text GLabel 3100 2900 2    50   Input ~ 0
+Col5
+Text GLabel 3100 4100 2    50   Input ~ 0
+Col11
+Text GLabel 3100 4200 2    50   Input ~ 0
+Col10
+Text GLabel 3100 4300 2    50   Input ~ 0
+Col9
+Text GLabel 3100 4400 2    50   Input ~ 0
+Col8
+Text GLabel 3100 4500 2    50   Input ~ 0
+Col7
+Text GLabel 3100 4600 2    50   Input ~ 0
+Col6
+Text GLabel 3100 3300 2    50   Input ~ 0
+Row0
+Text GLabel 3100 3500 2    50   Input ~ 0
+Row1
+Text GLabel 3100 3600 2    50   Input ~ 0
+Row2
+Text GLabel 3100 2100 2    50   Input ~ 0
+Row3
+Text GLabel 3100 2200 2    50   Input ~ 0
+Row4
 $EndSCHEMATC
